Commit message: refactor: update Modbus RTU communication to use single register writes and rename parameter arguments in SusGrip driver

File: susgrip_2f/susgrip_2f_description/urdf/susgrip_2f_macro.xacro (robot description, xacro)
@@ -183,5 +183,7 @@
         rpy="-1.570796 0. 0." />
       <geometry>
-        <cylinder radius="0.04" length="0.12" />
+        <mesh
+          filename="package://susgrip_2f_description/meshes/susgrip_2f_full/SUS_2F_Base.STL"
+          />
       </geometry>
     </collision>
@@ -209,5 +211,13 @@
       </material>
     </visual>
-    <!-- No collision -->
+    <collision>
+      <origin
+        xyz="0. 0. 0."
+        rpy="0. 0. 0." />
+      <geometry>
+        <mesh
+          filename="package://susgrip_2f_description/meshes/susgrip_2f_full/SUS_2F_Slider_L.obj"/>
+      </geometry>
+    </collision>
   </link>
   <joint
@@ -247,5 +257,13 @@
       </material>
     </visual>
-    <!-- No collision -->
+    <collision>
+      <origin
+        xyz="0.053 0. -0.043"
+        rpy="0. 0. 0." />
+      <geometry>
+        <mesh
+          filename="package://susgrip_2f_description/meshes/susgrip_2f_full/SUS_2F_Outer_L.obj"/>
+      </geometry>
+    </collision>
   </link>
   <joint
@@ -285,5 +303,13 @@
       </material>
     </visual>
-    <!-- No collision -->
+        <collision>
+      <origin
+        xyz="0.053 0 -0.097"
+        rpy="0 0 0" />
+      <geometry>
+        <mesh
+          filename="package://susgrip_2f_description/meshes/susgrip_2f_full/SUS_2F_Finger_L.obj"/>
+      </geometry>
+    </collision>
   </link>
   <joint
@@ -322,5 +348,13 @@
       </material>
     </visual>
-    <!-- No collision -->
+        <collision>
+      <origin
+        xyz="0.04 0. -0.097"
+        rpy="0. 0. 0." />
+      <geometry>
+        <mesh
+          filename="package://susgrip_2f_description/meshes/susgrip_2f_full/SUS_2F_Inner_L.obj"/>
+      </geometry>
+    </collision>
   </link>
   <joint
@@ -359,5 +393,13 @@
       </material>
     </visual>
-    <!-- No collision -->
+    <collision>
+      <origin
+        xyz="0. 0.016 0.027"
+        rpy="0. 0. -1.570796" />
+      <geometry>
+        <mesh
+          filename="package://susgrip_2f_description/meshes/susgrip_2f_full/SUS_2F_Pad_L.obj"/>
+      </geometry>
+    </collision>
   </link>
   <joint
@@ -397,5 +439,13 @@
       </material>
     </visual>
-    <!-- No collision -->
+    <collision>
+      <origin
+        xyz="0. -0.016 0.027"
+        rpy="0. 0. 1.570796" />
+      <geometry>
+        <mesh
+          filename="package://susgrip_2f_description/meshes/susgrip_2f_full/SUS_2F_Passive_Link_L.obj"/>
+      </geometry>
+    </collision>
   </link>
   <joint
@@ -437,5 +487,13 @@
       </material>
     </visual>
-    <!-- No collision -->
+    <collision>
+      <origin
+        xyz="0. 0. 0."
+        rpy="0. 0. 0." />
+      <geometry>
+        <mesh
+          filename="package://susgrip_2f_description/meshes/susgrip_2f_full/SUS_2F_Slider_R.obj"/>
+      </geometry>
+    </collision>
   </link>
   <joint
@@ -475,5 +533,13 @@
       </material>
     </visual>
-    <!-- No collision -->
+    <collision>
+      <origin
+        xyz="-0.053 0. -0.043"
+        rpy="0. 0. 3.141592" />
+      <geometry>
+        <mesh
+          filename="package://susgrip_2f_description/meshes/susgrip_2f_full/SUS_2F_Outer_R.obj"/>
+      </geometry>
+    </collision>
   </link>
   <joint
@@ -513,5 +579,13 @@
       </material>
     </visual>
-    <!-- No collision -->
+    <collision>
+      <origin
+        xyz="0.053 0 -0.097"
+        rpy="0 0 0" />
+      <geometry>
+        <mesh
+          filename="package://susgrip_2f_description/meshes/susgrip_2f_full/SUS_2F_Finger_R.obj"/>
+      </geometry>
+    </collision>
   </link>
   <joint
@@ -550,5 +624,13 @@
       </material>
     </visual>
-    <!-- No collision -->
+    <collision>
+      <origin
+        xyz="0.04 0. -0.097"
+        rpy="0. 0. 3.141592" />
+      <geometry>
+        <mesh
+          filename="package://susgrip_2f_description/meshes/susgrip_2f_full/SUS_2F_Inner_R.obj"/>
+      </geometry>
+    </collision>
   </link>
   <joint
@@ -587,5 +669,13 @@
       </material>
     </visual>
-    <!-- No collision -->
+    <collision>
+      <origin
+        xyz="0. -0.016 0.027"
+        rpy="0. 0. 1.570796" />
+      <geometry>
+        <mesh
+          filename="package://susgrip_2f_description/meshes/susgrip_2f_full/SUS_2F_Pad_R.obj"/>
+      </geometry>
+    </collision>
   </link>
   <joint
@@ -625,5 +715,13 @@
       </material>
     </visual>
-    <!-- No collision -->
+    <collision>
+      <origin
+        xyz="0. 0.016 0.027"
+        rpy="0. 0. -1.570796" />
+      <geometry>
+        <mesh
+          filename="package://susgrip_2f_description/meshes/susgrip_2f_full/SUS_2F_Passive_Link_R.obj"/>
+      </geometry>
+    </collision>
   </link>
   <joint
