Commit message: update damping and friction to run successfully gripper

File: install/susgrip_2f_gazebo/share/susgrip_2f_gazebo/urdf/susgrip_2f_gazebo.urdf.xacro (robot description, xacro)
@@ -4,6 +4,6 @@
         <xacro:property name="gripper_mass" value="1.0" />
         <xacro:property name="finger_mass" value="0.1" />
-        <xacro:property name="joint_damping" value="50.0" />
-        <xacro:property name="joint_friction" value="1.0" />
+        <xacro:property name="joint_damping" value="0.01" />
+        <xacro:property name="joint_friction" value="0.0" />
         <xacro:property name="joint_effort" value="100.0" />
         <xacro:property name="joint_velocity" value="0.05" />

File: src/susgrip_2f/susgrip_2f_gazebo/urdf/susgrip_2f_gazebo.urdf.xacro (robot description, xacro)
@@ -4,6 +4,6 @@
         <xacro:property name="gripper_mass" value="1.0" />
         <xacro:property name="finger_mass" value="0.1" />
-        <xacro:property name="joint_damping" value="0.1" />
-        <xacro:property name="joint_friction" value="0.1" />
+        <xacro:property name="joint_damping" value="0.01" />
+        <xacro:property name="joint_friction" value="0.0" />
         <xacro:property name="joint_effort" value="100.0" />
         <xacro:property name="joint_velocity" value="0.05" />
