Commit message: done urdf modification

File: src/susgrip_2f/susgrip_2f_gazebo/urdf/susgrip_2f_gazebo.urdf.xacro (robot description, xacro)
@@ -4,6 +4,6 @@
         <xacro:property name="gripper_mass" value="1.0" />
         <xacro:property name="finger_mass" value="0.1" />
-        <xacro:property name="joint_damping" value="50.0" />
-        <xacro:property name="joint_friction" value="1.0" />
+        <xacro:property name="joint_damping" value="0.1" />
+        <xacro:property name="joint_friction" value="0.1" />
         <xacro:property name="joint_effort" value="100.0" />
         <xacro:property name="joint_velocity" value="0.05" />

Commit message: improve gripper control and Cartesian object   handling

File: src/susgrip_2f/susgrip_2f_gazebo/urdf/susgrip_2f_gazebo.urdf.xacro (robot description, xacro)
@@ -8,5 +8,10 @@
         <xacro:property name="joint_effort" value="100.0" />
         <xacro:property name="joint_velocity" value="0.05" />
-        <xacro:property name="joint_limit_upper" value="0.065" />
+        <!--
+          The controller commands at most 0.065 m.  Leave 5 mm of physical
+          travel beyond that command limit so Gazebo never wedges the finger
+          exactly against the prismatic joint's hard stop.
+        -->
+        <xacro:property name="joint_limit_upper" value="0.070" />
         <material name="${prefix}color_base">
             <color rgba="0.423529 0.494118 0.882353 1.0" />
@@ -31,7 +36,8 @@
             </visual>
             <collision>
-                <origin xyz="0 0 0" rpy="0 0 0" />
+                <!-- Simple collision geometry keeps Gazebo physics fast. -->
+                <origin xyz="0 0 0.0615" rpy="0 0 0" />
                 <geometry>
-                    <mesh filename="package://susgrip_2f_description/meshes/susgrip_2f_simple/2F_MainBody.STL" />
+                    <cylinder radius="0.055" length="0.123" />
                 </geometry>
             </collision>
@@ -62,7 +68,7 @@
             </visual>
             <collision>
-                <origin xyz="0 0 0" rpy="0 0 0" />
+                <origin xyz="0 0 0.04" rpy="0 0 0" />
                 <geometry>
-                    <mesh filename="package://susgrip_2f_description/meshes/susgrip_2f_simple/FingerTip.STL" />
+                    <box size="0.016 0.020 0.080" />
                 </geometry>
             </collision>
@@ -77,6 +83,6 @@
             <mu1>2.0</mu1>
             <mu2>2.0</mu2>
-            <kp>1000000.0</kp>
-            <kd>100.0</kd>
+            <kp>100000.0</kp>
+            <kd>10.0</kd>
             <minDepth>0.002</minDepth>
             <maxVel>0.0</maxVel>
@@ -93,7 +99,7 @@
             </visual>
             <collision>
-                <origin xyz="0 0 0" rpy="0 0 0" />
+                <origin xyz="0 0 0.04" rpy="0 0 0" />
                 <geometry>
-                    <mesh filename="package://susgrip_2f_description/meshes/susgrip_2f_simple/FingerTip.STL" />
+                    <box size="0.016 0.020 0.080" />
                 </geometry>
             </collision>
@@ -108,6 +114,6 @@
             <mu1>2.0</mu1>
             <mu2>2.0</mu2>
-            <kp>1000000.0</kp>
-            <kd>100.0</kd>
+            <kp>100000.0</kp>
+            <kd>10.0</kd>
             <minDepth>0.002</minDepth>
             <maxVel>0.0</maxVel>

File: src/ur3_moveit_control/urdf/ur3_with_susgrip.urdf.xacro (robot description, xacro)
@@ -68,4 +68,18 @@
                 <state_interface name="effort"/>
             </joint>
+            <!--
+              Ignition ros2_control does not infer the simulated mimic joint
+              from the URDF <mimic> tag alone. Register the passive finger in
+              ros2_control so it follows the commanded gripper_joint.
+            -->
+            <joint name="gripper_joint_mimic">
+                <command_interface name="position">
+                    <param name="min">0.0</param>
+                    <param name="max">0.065</param>
+                </command_interface>
+                <state_interface name="position"/>
+                <state_interface name="velocity"/>
+                <state_interface name="effort"/>
+            </joint>
         </ros2_control>
         <!--
