Commit message: done side grasp

File: src/ur3_moveit_control/urdf/ur3_with_susgrip.urdf.xacro (robot description, xacro)
@@ -13,11 +13,12 @@
         <origin xyz="0 0 0.015" rpy="0 0 0" />
     </xacro:susgrip_2f_gazebo>
-    <!-- TCP at the center of the gripper opening. -->
-    <!-- gripper_body is 0.015 m from tool0; finger origins are at z=0.112 m. -->
+    <!-- TCP at the geometric center of the gripper opening. -->
+    <!-- Finger roots are at z=0.112 m and each finger is 0.080 m long, so -->
+    <!-- the grasp center is another 0.040 m along the gripper +Z axis. -->
     <link name="gripper_tcp"/>
     <joint name="gripper_tcp_joint" type="fixed">
         <parent link="gripper_body"/>
         <child link="gripper_tcp"/>
-        <origin xyz="0 0 0.112" rpy="0 0 0"/>
+        <origin xyz="0 0 0.152" rpy="0 0 0"/>
     </joint>
     <!-- 1. Eye-in-Hand Camera TF (from Calibration) -->
