Commit message: adding attach and lift code

File: install/ur3_moveit_control/share/ur3_moveit_control/urdf/ur3_with_susgrip.urdf.xacro (robot description, xacro)
@@ -13,4 +13,12 @@
         <origin xyz="0 0 0.015" rpy="0 0 0" />
     </xacro:susgrip_2f_gazebo>
+    <!-- TCP at the center of the gripper opening. -->
+    <!-- gripper_body is 0.015 m from tool0; finger origins are at z=0.112 m. -->
+    <link name="gripper_tcp"/>
+    <joint name="gripper_tcp_joint" type="fixed">
+        <parent link="gripper_body"/>
+        <child link="gripper_tcp"/>
+        <origin xyz="0 0 0.112" rpy="0 0 0"/>
+    </joint>
     <!-- 1. Eye-in-Hand Camera TF (from Calibration) -->
     <link name="camera_link"/>

File: install/ur_moveit_config/share/ur_moveit_config/srdf/ur3_with_susgrip.srdf.xacro (robot description, xacro)
@@ -6,5 +6,5 @@
   <xacro:arg name="prefix" default="" />
   <xacro:include filename="$(find ur_moveit_config)/srdf/ur_macro.srdf.xacro"/>
-  <xacro:ur_srdf name="$(arg name)" prefix="$(arg prefix)"/>
+  <xacro:ur_srdf name="$(arg name)" prefix="$(arg prefix)" tip_link="gripper_tcp"/>
   <!-- Gripper planning group -->
   <group name="gripper">

File: install/ur_moveit_config/share/ur_moveit_config/srdf/ur_macro.srdf.xacro (robot description, xacro)
@@ -5,5 +5,5 @@
     A URDF file must exist for this robot as well, where the joints and the links that are referenced are defined
 -->
-  <xacro:macro name="ur_srdf" params="name prefix">
+  <xacro:macro name="ur_srdf" params="name prefix tip_link:=tool0">
     <!--GROUPS - Representation of a set of joints and links. This can be useful for specifying DOF to plan for, defining arms, end effectors, etc-->
     <!--LINKS - When a link is specified, the parent joint of that link (if it exists) is automatically included-->
@@ -12,5 +12,5 @@
     <!--SUBGROUPS - Groups can also be formed by referencing to already defined group names-->
     <group name="${prefix}${name}_manipulator">
-      <chain base_link="${prefix}base_link" tip_link="${prefix}tool0" />
+      <chain base_link="${prefix}base_link" tip_link="${prefix}${tip_link}" />
     </group>
     <!--GROUP STATES - Purpose - Define a named state for a particular group, in terms of joint values. This is useful to define states like 'folded arms'-->

File: src/ur_simulation_gz/urdf/ur_gz.urdf.xacro (robot description, xacro)
@@ -59,5 +59,5 @@
     force_abs_paths="true"
     >
-    <origin xyz="0.3 0 0.825" rpy="0 0 0" />          <!-- position robot in the world -->
+    <origin xyz="0 0 0" rpy="0 0 0" />          <!-- position robot in the world -->
   </xacro:ur_robot>
   <gazebo reference="world">

Commit message: 3/8

File: install/ur3_moveit_control/share/ur3_moveit_control/urdf/ur3_with_susgrip.urdf.xacro (robot description, xacro)
@@ -1,72 +1 @@
-<?xml version="1.0"?>
-<robot xmlns:xacro="http://wiki.ros.org/xacro" name="$(arg name)">
-    <xacro:arg name="name" default="ur"/>
-    <xacro:arg name="sim_ignition" default="false"/>
-    <!-- Include the default UR robot xacro -->
-    <xacro:include filename="$(find ur_description)/urdf/ur.urdf.xacro"/>
-    <!-- Include the SusGrip 2F gripper xacro -->
-    <!-- The prefix and parent are needed to attach it correctly -->
-    <xacro:include filename="$(find susgrip_2f_gazebo)/urdf/susgrip_2f_gazebo.urdf.xacro"/>
-    <!-- Attach the gripper to the tool0 link of the UR robot -->
-    <!-- Thêm khoảng cách 1.5 cm (0.015 m) dọc theo trục Z -->
-    <xacro:susgrip_2f_gazebo prefix="" parent="tool0">
-        <origin xyz="0 0 0.015" rpy="0 0 0" />
-    </xacro:susgrip_2f_gazebo>
-    <!-- TCP at the center of the gripper opening. -->
-    <!-- gripper_body is 0.015 m from tool0; finger origins are at z=0.112 m. -->
-    <link name="gripper_tcp"/>
-    <joint name="gripper_tcp_joint" type="fixed">
-        <parent link="gripper_body"/>
-        <child link="gripper_tcp"/>
-        <origin xyz="0 0 0.112" rpy="0 0 0"/>
-    </joint>
-    <!-- 1. Eye-in-Hand Camera TF (from Calibration) -->
-    <link name="camera_link"/>
-    <joint name="camera_fixed_joint" type="fixed">
-        <parent link="tool0"/>
-        <child link="camera_link"/>
-        <origin xyz="0.001623 -0.106306 0.013148" rpy="0.163640 -1.535191 1.364251"/>
-    </joint>
-    <!-- 2. Spacer Cylinder between tool0 and Gripper -->
-    <!-- Bán kính 5cm (0.05m), Độ dày 1.5cm (0.015m) -->
-    <link name="spacer_cylinder">
-        <visual>
-            <geometry>
-                <cylinder radius="0.05" length="0.015"/>
-            </geometry>
-            <material name="gray">
-                <color rgba="0.5 0.5 0.5 1.0"/>
-            </material>
-        </visual>
-        <collision>
-            <geometry>
-                <cylinder radius="0.05" length="0.015"/>
-            </geometry>
-        </collision>
-    </link>
-    <joint name="spacer_joint" type="fixed">
-        <parent link="tool0"/>
-        <child link="spacer_cylinder"/>
-        <!-- Đặt tâm của hình trụ vào giữa khoảng trống (0.015 / 2 = 0.0075) -->
-        <origin xyz="0 0 0.0075" rpy="0 0 0"/>
-    </joint>
-    <!-- 3. Gazebo ROS 2 Control for Gripper (Only if sim_ignition:=true) -->
-    <xacro:if value="$(arg sim_ignition)">
-        <ros2_control name="SusGripGazeboSystem" type="system">
-            <hardware>
-                <plugin>ign_ros2_control/IgnitionSystem</plugin>
-            </hardware>
-            <joint name="gripper_joint">
-                <command_interface name="position">
-                    <param name="min">0.0</param>
-                    <param name="max">0.065</param>
-                </command_interface>
-                <state_interface name="position">
-                    <param name="initial_value">0.0</param>
-                </state_interface>
-                <state_interface name="velocity"/>
-                <state_interface name="effort"/>
-            </joint>
-        </ros2_control>
-    </xacro:if>
-</robot>
+/home/com9/uet_ws/src/ur3_moveit_control/urdf/ur3_with_susgrip.urdf.xacro

File: install/ur3_moveit_control/share/ur3_moveit_control/urdf/ur3_with_susgrip_gazebo.urdf.xacro (robot description, xacro)
@@ -1,6 +1 @@
-<?xml version="1.0"?>
-<robot xmlns:xacro="http://wiki.ros.org/xacro" name="$(arg name)">
-    <xacro:arg name="name" default="ur"/>
-    <xacro:arg name="sim_gazebo" default="true"/>
-    <xacro:include filename="$(find ur3_moveit_control)/urdf/ur3_with_susgrip.urdf.xacro"/>
-</robot>
+/home/com9/uet_ws/src/ur3_moveit_control/urdf/ur3_with_susgrip_gazebo.urdf.xacro

File: src/ur3_moveit_control/urdf/ur3_with_susgrip.urdf.xacro (robot description, xacro)
@@ -88,9 +88,13 @@
           cannot make pick_box follow the gripper.  This system creates/removes
           a real fixed joint when Empty messages arrive on the topics below.
+          gripper_tcp and gripper_body are connected through fixed joints.
+          Gazebo collapses both frames into wrist_3_link while converting the
+          URDF to SDF; the two movable finger links are re-parented to it.
+          DetachableJoint must therefore use the surviving physical link name.
         -->
         <gazebo>
             <plugin filename="ignition-gazebo-detachable-joint-system"
                     name="ignition::gazebo::systems::DetachableJoint">
-                <parent_link>gripper_tcp</parent_link>
+                <parent_link>wrist_3_link</parent_link>
                 <child_model>pick_box</child_model>
                 <child_link>box_link</child_link>
